File: kicad/mcupcb_30pins.kicad_sch (KiCad schematic)
At the start: 34 parts

Commit message: Fixed flipped D+/D-
Parts:
- C1, C2: value (none) -> 10p; footprint (none) -> Capacitor_SMD:C_0603_1608Metric
- C10, C3, C4, C7, C8, C9: value (none) -> 0.1u; footprint (none) -> Capacitor_SMD:C_0603_1608Metric
- C5, C6: value (none) -> 1u; footprint (none) -> Capacitor_SMD:C_0805_2012Metric
- D1: value (none) -> PRTR5V0U2X; footprint (none) -> Package_TO_SOT_SMD:SOT-143
- F1: value (none) -> Polyfuse; footprint (none) -> Fuse:Fuse_1206_3216Metric
- H1, H2, H3: value (none) -> MountingHole; footprint (none) -> MCUPCB_footprints:MountingHole_M2_NoCu
- H10, H9: value (none) -> MountingHole; footprint (none) -> MCUPCB_footprints:Breakaway_panel
- H4: value (none) -> MountingHole; footprint (none) -> MCUPCB_footprints:MountingHole_M2_PTH
- H5, H6, H7: value (none) -> MountingHole; footprint (none) -> MCUPCB_footprints:Breakaway_small
- H8: value (none) -> MountingHole; footprint (none) -> Symbol:OSHW-Logo_5.7x6mm_SilkScreen
- J1: value (none) -> Conn_01x30_MountingPin; footprint (none) -> Connector_FFC-FPC:Hirose_FH12-30S-0.5SH_1x30-1MP_P0.50mm_Horizontal
- J2: value (none) -> ICSP; footprint (none) -> MCUPCB_footprints:Tag-Connect_TC2030-IDC-NL_2x03_P1.27mm_Vertical
- R1: value (none) -> 10k; footprint (none) -> Resistor_SMD:R_0603_1608Metric
- R2, R3: value (none) -> 5.1k; footprint (none) -> Resistor_SMD:R_0603_1608Metric
- R4, R5: value (none) -> 22; footprint (none) -> Resistor_SMD:R_0603_1608Metric
- TP1, TP2: value (none) -> TestPoint; footprint (none) -> TestPoint:TestPoint_Pad_D1.5mm
- U1: value (none) -> ATmega32U4-AU; footprint (none) -> Package_QFP:TQFP-44_10x10mm_P0.8mm
- USB1: value (none) -> HRO-TYPE-C-31-M-12; footprint (none) -> Connector_USB:USB_C_Receptacle_HRO_TYPE-C-31-M-12
- Y1: value (none) -> X322516MLB4SI; footprint (none) -> Crystal:Crystal_SMD_3225-4Pin_3.2x2.5mm
Connections:
- net D+: now also D1.3 (I/O2), R4.2; no longer D1.2 (I/O1), R5.2
- net D-: now also D1.2 (I/O1), R5.2; no longer D1.3 (I/O2), R4.2
